Commit message: messhes parse

File: urdf2/mr_robot.urdf (robot description, URDF)
Before this commit: robot mr_robot, 7 links, 6 joints
Links:
- link Lidar_1: geometry collision mesh filename=/home/vansh/intern-ardee/src/fcl-cpp/meshes/Lidar_1.stl scale=0.001 0.001 0.001; visual mesh filename=/home/vansh/intern-ardee/src/fcl-cpp /meshes/Lidar_1.stl scale=0.001 0.001 0.001
- link base_link: geometry collision mesh filename=/home/vansh/intern-ardee/src/fcl-cpp/meshes/base_link.stl scale=0.001 0.001 0.001; visual mesh filename=/home/vansh/intern-ardee/src/fcl-cpp/meshes/base_link.stl scale=0.001 0.001 0.001
- link gps_1: geometry collision mesh filename=/home/vansh/intern-ardee/src/fcl-cpp/meshes/gps_1.stl scale=0.001 0.001 0.001; visual mesh filename=/home/vansh/intern-ardee/src/fcl-cpp/meshes/gps_1.stl scale=0.001 0.001 0.001
- link imu_1: geometry collision mesh filename=/home/vansh/intern-ardee/src/fcl-cpp/meshes/imu_1.stl scale=0.001 0.001 0.001; visual mesh filename=/home/vansh/intern-ardee/src/fcl-cpp/meshes/imu_1.stl scale=0.001 0.001 0.001
- link left_wheel_1: geometry collision mesh filename=/home/vansh/intern-ardee/src/fcl-cpp/meshes/left_wheel_1.stl scale=0.001 0.001 0.001; visual mesh filename=/home/vansh/intern-ardee/src/fcl-cpp/meshes/left_wheel_1.stl scale=0.001 0.001 0.001
- link right_wheel__1: geometry collision mesh filename=/home/vansh/intern-ardee/src/fcl-cpp/meshes/right_wheel__1.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 scale=0.001 0.001 0.001; visual mesh filename=/home/vansh/intern-ardee/src/fcl-cpp/meshes/right_wheel__1.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 scale=0.001 0.001 0.001
Joints:
- joint left_motor_joint: axis -0.0 1.0 0.0 -> -0.0 -0.4 0.0; origin xyz=0.0 0.181075 -0.0556 rpy=0 0 0 -> xyz=0.0 -0.4 0.0 rpy=0 0.0 0
